Commit message: feat: add ros2 bridge interface

File: resource/RobotisOp3.urdf (robot description, URDF)
Before this commit: robot /home/haze/Desktop/RobotisOp3.urdf, 30 links, 29 joints
Links:
- removed link Accelerometer
- removed link AnkleLSolid
- removed link AnkleRSolid
- removed link ArmLowerLbowSolid
- removed link ArmLowerRbowSolid
- removed link ArmUpperLSolid
- removed link ArmUpperRSolid
- removed link BodyLed
- removed link Camera
- removed link FootLSolid
- removed link FootRSolid
- removed link Gyro
- removed link HeadLed
- removed link HeadSolid
- removed link LegLowerLSolid
- removed link LegLowerRSolid
- removed link LegUpperLSolid
- removed link LegUpperRSolid
- removed link NeckSolid
- removed link PelvLSolid
- removed link PelvRSolid
- removed link PelvYLSolid
- removed link PelvYRSolid
- removed link ShoulderLSolid
- removed link ShoulderRSolid
- removed link Speaker
- removed link appearance
- removed link appearance_0
- removed link base_link
- removed link body
Joints:
- removed joint AnkleL
- removed joint AnkleR
- removed joint ArmLowerL
- removed joint ArmLowerR
- removed joint ArmUpperL
- removed joint ArmUpperR
- removed joint BodyLed_appearance_0_joint
- removed joint FootL
- removed joint FootR
- removed joint Head
- removed joint HeadLed_appearance_joint
- removed joint HeadSolid_Camera_joint
- removed joint HeadSolid_HeadLed_joint
- removed joint LegLowerL
- removed joint LegLowerR
- removed joint LegUpperL
- removed joint LegUpperR
- removed joint Neck
- removed joint PelvL
- removed joint PelvR
- removed joint PelvYL
- removed joint PelvYR
- removed joint ShoulderL
- removed joint ShoulderR
- removed joint base_link_Accelerometer_joint
- removed joint base_link_BodyLed_joint
- removed joint base_link_Gyro_joint
- removed joint base_link_Speaker_joint
- removed joint base_link_body_joint
